Commit message: Update jackal_rplidar_vr.urdf.xacro
rplidar --> hokuyo

for outdoor

File: urdf/jackal_rplidar_vr.urdf.xacro (robot description, xacro)
@@ -218,34 +218,34 @@
     <origin xyz="${mount_spacing} 0 0" />
   </joint>
-  <!-- RPLidar Link -->
-  <link name="rplidar_link">
-    <visual>
-      <origin xyz="0 0 0" rpy="0 0 0"/>
-      <geometry>
-        <cylinder length="0.060" radius="0.050"/>
-      </geometry>
-      <material name="black" />
-    </visual>
-    <collision>
-      <origin xyz="0 0 0" rpy="0 0 0"/>
-      <geometry>
-        <cylinder length="0.060" radius="0.050"/>
-      </geometry>
-    </collision>
-    <inertial>
-      <origin xyz="0 0 0" rpy="0 0 0"/>
-      <mass value="0.4"/>
-      <inertia
-        ixx="0.0008" ixy="0" ixz="0"
-        iyy="0.0008" iyz="0"
-        izz="0.0008"/>
-    </inertial>
-  </link>
-  <!-- RPLidar Joint -->
-  <joint name="rplidar_joint" type="fixed">
-    <origin xyz="0 0 0.1" rpy="0 0 0" />
-    <parent link="rear_mount" />
-    <child link="rplidar_link" />
-  </joint>
+<!-- Hokuyo Link -->
+<link name="hokuyo_link">
+  <visual>
+    <origin xyz="0 0 0" rpy="0 0 0"/>
+    <geometry>
+      <box size="0.10 0.10 0.10"/>
+    </geometry>
+    <material name="black" />
+  </visual>
+  <collision>
+    <origin xyz="0 0 0" rpy="0 0 0"/>
+    <geometry>
+      <box size="0.10 0.10 0.10"/>
+    </geometry>
+  </collision>
+  <inertial>
+    <origin xyz="0 0 0" rpy="0 0 0"/>
+    <mass value="0.1"/>
+    <inertia
+      ixx="0.0001" ixy="0" ixz="0"
+      iyy="0.0001" iyz="0"
+      izz="0.0001"/>
+  </inertial>
+</link>
+<!-- Hokuyo Joint -->
+<joint name="hokuyo_joint" type="fixed">
+  <origin xyz="0 0 0.1" rpy="0 0 0" />
+  <parent link="rear_mount" />
+  <child link="hokuyo_link" />
+</joint>
 <!-- Intel Realsense Camera Link -->
 <link name="realsense_camera_link">
